Commit message: 改了好多

File: src/rover_description/urdf/rover.xacro (robot description, xacro)
@@ -2,6 +2,4 @@
 <robot name="rover" xmlns:xacro="http://www.ros.org/wiki/xacro">
     <!-- ================= 1. 参数定义 ================= -->
-    <xacro:property name="length_wheel" value="0.05" />
-    <xacro:property name="radius_wheel" value="0.09" />
     <xacro:property name="PI" value="3.1415926"/>
     <!-- 车身尺寸 -->
@@ -9,34 +7,36 @@
     <xacro:property name="body_width" value="0.25"/>
     <xacro:property name="body_height" value="0.13"/>
+    <!-- 车轮尺寸 -->
+    <xacro:property name="length_wheel" value="0.05"/>
+    <xacro:property name="radius_wheel" value="0.09" />
     <!-- 轮子位置参数 -->
     <xacro:property name="wheel_offset_x" value="0.15"/>
     <xacro:property name="wheel_offset_y" value="0.16"/>
-    <!-- 摩擦力 (0.2 保证能转向) -->
+    <!-- 摩擦力 (后轮保持 0.2 提供抓地力，前轮后面单独设为 0) -->
     <xacro:property name="wheel_mu" value="0.2"/>
     <!-- ================= 2. 惯性矩阵计算 ================= -->
-    <xacro:macro name="default_inertial" params="mass">
+    <xacro:macro name="box_inertial" params="m x y z">
         <inertial>
-            <mass value="${mass}" />
-            <inertia ixx="${mass/12*(body_width*body_width + body_height*body_height)}" ixy="0.0" ixz="0.0"
-                     iyy="${mass/12*(body_len*body_len + body_height*body_height)}" iyz="0.0"
-                     izz="${mass/12*(body_len*body_len + body_width*body_width)}" />
+            <mass value="${m}"/>
+            <inertia ixx="${m*(y*y+z*z)/12}" ixy="0" ixz="0"
+                     iyy="${m*(x*x+z*z)/12}" iyz="0"
+                     izz="${m*(x*x+y*y)/12}" />
         </inertial>
     </xacro:macro>
-    <xacro:macro name="wheel_inertial" params="mass">
+    <xacro:macro name="cylinder_inertial" params="m r h">
         <inertial>
-            <mass value="${mass}" />
-            <inertia ixx="0.001" ixy="0.0" ixz="0.0" iyy="0.001" iyz="0.0" izz="0.001" />
+            <mass value="${m}"/>
+            <inertia ixx="${m*(3*r*r+h*h)/12}" ixy="0" ixz="0"
+                     iyy="${m*(3*r*r+h*h)/12}" iyz="0"
+                     izz="${m*r*r/2}" />
         </inertial>
     </xacro:macro>
     <!-- ================= 3. 机器人主体 ================= -->
-    <!-- Base Footprint -->
     <link name="base_footprint">
         <visual>
-            <geometry>
-                <box size="0.001 0.001 0.001"/>
-            </geometry>
-            <origin rpy="0 0 0" xyz="0 0 0"/>
-        </visual>
-        <xacro:default_inertial mass="0.0001"/>
+            <geometry><box size="0.001 0.001 0.001"/></geometry>
+            <origin rpy="0 0 0" xyz="0 0 0"/>
+        </visual>
+        <xacro:box_inertial m="5.0" x="0.001" y="0.001" z="0.001"/>
     </link>
     <joint name="base_footprint_joint" type="fixed">
@@ -45,118 +45,93 @@
         <child link="base_link" />
     </joint>
-    <!-- Base Link -->
     <link name="base_link">
         <visual>
+            <geometry><box size="${body_len} ${body_width} ${body_height}"/></geometry>
+            <origin rpy="0 0 0" xyz="0 0 0"/>
+            <material name="white"><color rgba="0.8 0.8 0.8 1"/></material>
+        </visual>
+        <collision>
+            <geometry><box size="${body_len} ${body_width} ${body_height}"/></geometry>
+            <origin rpy="0 0 0" xyz="0 0 0"/>
+        </collision>
+        <xacro:box_inertial m="5.0" x="${body_len}" y="${body_width}" z="${body_height}"/>
+    </link>
+    <!-- ================= 4. 四个轮子 ================= -->
+    <!-- [1] 前左轮 (Front Left) - 从动轮 -->
+    <link name="wheel_FL">
+        <visual>
             <geometry>
-                <box size="${body_len} ${body_width} ${body_height}"/>
+                <cylinder length="${length_wheel}" radius="${radius_wheel}"/>
             </geometry>
             <origin rpy="0 0 0" xyz="0 0 0"/>
-            <material name="white">
-                <color rgba="0.8 0.8 0.8 1"/>
-            </material>
-        </visual>
-        <collision>
-            <geometry>
-                <box size="${body_len} ${body_width} ${body_height}"/>
-            </geometry>
-            <origin rpy="0 0 0" xyz="0 0 0"/>
-        </collision>
-        <xacro:default_inertial mass="5.0"/>
-    </link>
-    <!-- ================= 4. 四个轮子 ================= -->
-    <!-- [1] 前左轮 (Front Left) -->
-    <link name="wheel_FL">
-        <visual>
-            <geometry><cylinder length="${length_wheel}" radius="${radius_wheel}"/></geometry>
-            <material name="black"><color rgba="0.1 0.1 0.1 1"/></material>
-        </visual>
-        <collision>
-            <geometry><cylinder length="${length_wheel}" radius="${radius_wheel}"/></geometry>
-        </collision>
-        <visual>
-            <geometry><cylinder length="0.06" radius="0.015"/></geometry>
-            <origin rpy="0 0 0" xyz="0 0 -0.03"/>
-            <material name="grey"><color rgba="0.5 0.5 0.5 1"/></material>
-        </visual>
+            <material name="black"><color rgba="0.1 0.1 0.1 1"/></material>
+        </visual>
+        <collision>
+            <geometry><cylinder length="${length_wheel}" radius="${radius_wheel}"/></geometry>
+            <origin rpy="0 0 0" xyz="0 0 0"/>
+        </collision>
+        <xacro:cylinder_inertial m="0.5" r="${radius_wheel}" h="${length_wheel}"/>
+    </link>
+    <joint name="joint_FL" type="continuous">
+        <parent link="base_link"/>
+        <child link="wheel_FL"/>
+        <origin rpy="${-PI/2} 0 0" xyz="${wheel_offset_x} ${wheel_offset_y} -0.02"/>
+        <axis xyz="0 0 1" />
+    </joint>
+    <!-- [2] 前右轮 (Front Right) - 从动轮 -->
+    <link name="wheel_FR">
+        <visual>
+            <geometry><cylinder length="${length_wheel}" radius="${radius_wheel}"/></geometry>
+            <origin rpy="0 0 0" xyz="0 0 0"/>
+            <material name="black"><color rgba="0.1 0.1 0.1 1"/></material>
+        </visual>
+        <collision>
+            <geometry><cylinder length="${length_wheel}" radius="${radius_wheel}"/></geometry>
+            <origin rpy="0 0 0" xyz="0 0 0"/>
+        </collision>
+        <xacro:cylinder_inertial m="0.5" r="${radius_wheel}" h="${length_wheel}"/>
+    </link>
+    <joint name="joint_FR" type="continuous">
+        <parent link="base_link"/>
+        <child link="wheel_FR"/>
+        <origin rpy="${-PI/2} 0 0" xyz="${wheel_offset_x} -${wheel_offset_y} -0.02"/>
+        <axis xyz="0 0 1" />
+    </joint>
+    <!-- [3] 后左轮 (Rear Left) - 驱动轮 -->
+    <link name="wheel_RL">
+        <visual>
+            <geometry><cylinder length="${length_wheel}" radius="${radius_wheel}"/></geometry>
+            <origin rpy="0 0 0" xyz="0 0 0"/>
+            <material name="black"><color rgba="0.1 0.1 0.1 1"/></material>
+        </visual>
+        <collision>
+            <geometry><cylinder length="${length_wheel}" radius="${radius_wheel}"/></geometry>
+            <origin rpy="0 0 0" xyz="0 0 0"/>
+        </collision>
         <mu1>${wheel_mu}</mu1>
         <mu2>${wheel_mu}</mu2>
-        <xacro:wheel_inertial mass="0.5"/>
-    </link>
-    <!-- ⚠️ 关键修改：前轮改为 FIXED，解决 RViz 不显示问题 -->
-    <joint name="joint_FL" type="fixed">
-        <parent link="base_link"/>
-        <child link="wheel_FL"/>
-        <origin rpy="${-PI/2} 0 0" xyz="${wheel_offset_x} ${wheel_offset_y} -0.02"/>
-        <axis xyz="0 0 1" />
-    </joint>
-    <!-- [2] 前右轮 (Front Right) -->
-    <link name="wheel_FR">
-        <visual>
-            <geometry><cylinder length="${length_wheel}" radius="${radius_wheel}"/></geometry>
-            <material name="black"><color rgba="0.1 0.1 0.1 1"/></material>
-        </visual>
-        <collision>
-            <geometry><cylinder length="${length_wheel}" radius="${radius_wheel}"/></geometry>
-        </collision>
-        <visual>
-            <geometry><cylinder length="0.06" radius="0.015"/></geometry>
-            <origin rpy="0 0 0" xyz="0 0 0.03"/>
-            <material name="grey"><color rgba="0.5 0.5 0.5 1"/></material>
-        </visual>
+        <xacro:cylinder_inertial m="0.5" r="${radius_wheel}" h="${length_wheel}"/>
+    </link>
+    <joint name="joint_RL" type="continuous">
+        <parent link="base_link"/>
+        <child link="wheel_RL"/>
+        <origin rpy="${-PI/2} 0 0" xyz="-${wheel_offset_x} ${wheel_offset_y} -0.02"/>
+        <axis xyz="0 0 1" />
+    </joint>
+    <!-- [4] 后右轮 (Rear Right) - 驱动轮 (你漏了这部分！帮你补上了) -->
+    <link name="wheel_RR">
+        <visual>
+            <geometry><cylinder length="${length_wheel}" radius="${radius_wheel}"/></geometry>
+            <origin rpy="0 0 0" xyz="0 0 0"/>
+            <material name="black"><color rgba="0.1 0.1 0.1 1"/></material>
+        </visual>
+        <collision>
+            <geometry><cylinder length="${length_wheel}" radius="${radius_wheel}"/></geometry>
+            <origin rpy="0 0 0" xyz="0 0 0"/>
+        </collision>
         <mu1>${wheel_mu}</mu1>
         <mu2>${wheel_mu}</mu2>
-        <xacro:wheel_inertial mass="0.5"/>
-    </link>
-    <!-- ⚠️ 关键修改：前轮改为 FIXED -->
-    <joint name="joint_FR" type="fixed">
-        <parent link="base_link"/>
-        <child link="wheel_FR"/>
-        <origin rpy="${-PI/2} 0 0" xyz="${wheel_offset_x} -${wheel_offset_y} -0.02"/>
-        <axis xyz="0 0 1" />
-    </joint>
-    <!-- [3] 后左轮 (Rear Left) - 驱动轮 -->
-    <link name="wheel_RL">
-        <visual>
-            <geometry><cylinder length="${length_wheel}" radius="${radius_wheel}"/></geometry>
-            <material name="black"><color rgba="0.1 0.1 0.1 1"/></material>
-        </visual>
-        <collision>
-            <geometry><cylinder length="${length_wheel}" radius="${radius_wheel}"/></geometry>
-        </collision>
-        <visual>
-            <geometry><cylinder length="0.06" radius="0.015"/></geometry>
-            <origin rpy="0 0 0" xyz="0 0 -0.03"/>
-            <material name="grey"><color rgba="0.5 0.5 0.5 1"/></material>
-        </visual>
-        <mu1>${wheel_mu}</mu1>
-        <mu2>${wheel_mu}</mu2>
-        <xacro:wheel_inertial mass="0.5"/>
-    </link>
-    <!-- 保持 continuous，因为它是驱动轮 -->
-    <joint name="joint_RL" type="continuous">
-        <parent link="base_link"/>
-        <child link="wheel_RL"/>
-        <origin rpy="${-PI/2} 0 0" xyz="-${wheel_offset_x} ${wheel_offset_y} -0.02"/>
-        <axis xyz="0 0 1" />
-    </joint>
-    <!-- [4] 后右轮 (Rear Right) - 驱动轮 -->
-    <link name="wheel_RR">
-        <visual>
-            <geometry><cylinder length="${length_wheel}" radius="${radius_wheel}"/></geometry>
-            <material name="black"><color rgba="0.1 0.1 0.1 1"/></material>
-        </visual>
-        <collision>
-            <geometry><cylinder length="${length_wheel}" radius="${radius_wheel}"/></geometry>
-        </collision>
-        <visual>
-            <geometry><cylinder length="0.06" radius="0.015"/></geometry>
-            <origin rpy="0 0 0" xyz="0 0 0.03"/>
-            <material name="grey"><color rgba="0.5 0.5 0.5 1"/></material>
-        </visual>
-        <mu1>${wheel_mu}</mu1>
-        <mu2>${wheel_mu}</mu2>
-        <xacro:wheel_inertial mass="0.5"/>
-    </link>
-    <!-- 保持 continuous，因为它是驱动轮 -->
+        <xacro:cylinder_inertial m="0.5" r="${radius_wheel}" h="${length_wheel}"/>
+    </link>
     <joint name="joint_RR" type="continuous">
         <parent link="base_link"/>
@@ -166,27 +141,5 @@
     </joint>
     <!-- ================= 5. 传感器 ================= -->
-    <!-- IMU -->
-    <joint name="imu_joint" type="fixed">
-        <axis xyz="0 1 0" />
-        <origin xyz="0.0 0 0.08" rpy="0 0 0"/>
-        <parent link="base_link"/>
-        <child link="imu_link"/>
-    </joint>
-    <link name="imu_link">
-        <visual>
-            <geometry><box size="0.05 0.05 0.02"/></geometry>
-            <material name="green"><color rgba="0 1 0 1"/></material>
-        </visual>
-        <inertial>
-            <mass value="0.01" />
-            <inertia ixx="1e-6" ixy="0" ixz="0" iyy="1e-6" iyz="0" izz="1e-6" />
-        </inertial>
-    </link>
-    <!-- 雷达支架 -->
-    <joint name="laserholder_joint" type="fixed">
-        <origin xyz="0.1 0.0 0.065" rpy="0 0 0"/>
-        <parent link="base_link"/>
-        <child link="laserholder_link"/>
-    </joint>
+    <!-- 1. 雷达支架 (Link + Joint) -->
     <link name="laserholder_link">
         <visual>
@@ -195,44 +148,29 @@
             <origin rpy="0 0 0" xyz="0 0 0.05"/>
         </visual>
-        <xacro:default_inertial mass="0.01"/>
+        <xacro:box_inertial m="0.01" x="0.02" y="0.02" z="0.1"/>
+    </link>
+    <joint name="laserholder_joint" type="fixed">
+        <origin xyz="0.1 0.0 0.065" rpy="0 0 0"/> <!-- 装在车头上方 -->
+        <parent link="base_link"/>
+        <child link="laserholder_link"/>
+    </joint>
+    <!-- 2. 雷达本体 (Link + Joint) -->
+    <link name="scan_link">
+        <visual>
+            <geometry><cylinder length="0.04" radius="0.04"/></geometry>
+            <material name="blue"><color rgba="0 0 1 1"/></material>
+        </visual>
+        <xacro:cylinder_inertial m="0.1" r="0.04" h="0.04"/>
     </link>
     <joint name="laser_joint" type="fixed">
-        <origin xyz="0.0 0.0 0.1" rpy="0 0 0"/>
+        <origin xyz="0.0 0.0 0.1" rpy="0 0 0"/> <!-- 装在支架顶上 -->
         <parent link="laserholder_link"/>
         <child link="scan_link"/>
     </joint>
-    <link name="scan_link">
-        <visual>
-            <geometry><cylinder length="0.04" radius="0.04"/></geometry>
-            <material name="blue"><color rgba="0 0 1 1"/></material>
-        </visual>
-        <xacro:default_inertial mass="0.1"/>
-    </link>
-    <!-- ================= 6. Gazebo 插件 ================= -->
-    <gazebo>
-        <plugin name='diff_drive' filename='libgazebo_ros_diff_drive.so'>
-            <ros>
-                <namespace>/</namespace>
-                <remapping>cmd_vel:=cmd_vel</remapping>
-                <remapping>odom:=odom</remapping>
-            </ros>
-            <!-- 驱动后轮 -->
-            <left_joint>joint_RL</left_joint>
-            <right_joint>joint_RR</right_joint>
-            <wheel_separation>${wheel_offset_y * 2}</wheel_separation>
-            <wheel_diameter>${radius_wheel * 2}</wheel_diameter>
-            <max_wheel_torque>100</max_wheel_torque>
-            <max_wheel_acceleration>2.0</max_wheel_acceleration>
-            <publish_odom>true</publish_odom>
-            <publish_odom_tf>true</publish_odom_tf>
-            <publish_wheel_tf>true</publish_wheel_tf>
-            <odometry_frame>odom</odometry_frame>
-            <robot_base_frame>base_footprint</robot_base_frame>
-        </plugin>
-    </gazebo>
+    <!-- 3. 雷达 Gazebo 插件 (刚才给你的修复版) -->
     <gazebo reference="scan_link">
         <sensor name="lidar" type="ray">
             <always_on>true</always_on>
-            <visualize>false</visualize>
+            <visualize>true</visualize>
             <update_rate>10</update_rate>
             <ray>
@@ -247,6 +185,6 @@
                 <range>
                     <min>0.120000</min>
-                    <max>8.0</max>
-                    <resolution>0.015000</resolution>
+                    <max>10.0</max>
+                    <resolution>0.02</resolution>
                 </range>
                 <noise>
@@ -265,30 +203,55 @@
         </sensor>
     </gazebo>
-    <gazebo reference="imu_link">
-        <gravity>true</gravity>
-        <sensor name="imu_sensor" type="imu">
-            <always_on>true</always_on>
-            <update_rate>100</update_rate>
-            <visualize>true</visualize>
-            <plugin filename="libgazebo_ros_imu_sensor.so" name="imu_plugin">
-                <topicName>imu</topicName>
-                <bodyName>imu_link</bodyName>
-                <updateRateHz>100.0</updateRateHz>
-                <gaussianNoise>0.0</gaussianNoise>
-                <xyzOffset>0 0 0</xyzOffset>
-                <rpyOffset>0 0 0</rpyOffset>
-                <frameName>imu_link</frameName>
-                <initialOrientationAsReference>false</initialOrientationAsReference>
-                <ros>
-                    <namespace>/</namespace>
-                    <remapping>~/out:=imu/data</remapping>
-                </ros>
-            </plugin>
-        </sensor>
-    </gazebo>
-    <gazebo reference="base_link"><material>Gazebo/White</material></gazebo>
-    <gazebo reference="wheel_FL"><material>Gazebo/Black</material></gazebo>
-    <gazebo reference="wheel_FR"><material>Gazebo/Black</material></gazebo>
+    <!-- ================= 6. Gazebo 物理属性 & 插件 ================= -->
+    <!-- ⚠️ 关键修正：给前轮设置零摩擦，模拟万向轮，否则转不动！ -->
+    <gazebo reference="wheel_FL">
+        <mu1>0.001</mu1> <mu2>0.001</mu2> <!-- 像冰一样滑 -->
+        <material>Gazebo/Black</material>
+    </gazebo>
+    <gazebo reference="wheel_FR">
+        <mu1>0.001</mu1> <mu2>0.001</mu2>
+        <material>Gazebo/Black</material>
+    </gazebo>
+    <!-- 后轮保持有摩擦，提供动力 -->
     <gazebo reference="wheel_RL"><material>Gazebo/Black</material></gazebo>
     <gazebo reference="wheel_RR"><material>Gazebo/Black</material></gazebo>
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
Commit message: 加了B样条

File: src/rover_description/urdf/rover.xacro (robot description, xacro)
@@ -119,5 +119,5 @@
         <axis xyz="0 0 1" />
     </joint>
-    <!-- [4] 后右轮 (Rear Right) - 驱动轮 (你漏了这部分！帮你补上了) -->
+    <!-- [4] 后右轮 (Rear Right) - 驱动轮 -->
     <link name="wheel_RR">
         <visual>
@@ -151,5 +151,5 @@
     </link>
     <joint name="laserholder_joint" type="fixed">
-        <origin xyz="0.1 0.0 0.065" rpy="0 0 0"/> <!-- 装在车头上方 -->
+        <origin xyz="0.1 0.0 0.065" rpy="0 0 0"/>
         <parent link="base_link"/>
         <child link="laserholder_link"/>
@@ -205,9 +205,11 @@
     <!-- ================= 6. Gazebo 物理属性 & 插件 ================= -->
     <gazebo reference="wheel_FL">
-        <mu1>0.001</mu1> <mu2>0.001</mu2> <!-- 像冰一样滑 -->
+        <mu1>0.5</mu1>
+        <mu2>0.001</mu2>
         <material>Gazebo/Black</material>
     </gazebo>
     <gazebo reference="wheel_FR">
-        <mu1>0.001</mu1> <mu2>0.001</mu2>
+        <mu1>0.5</mu1>
+        <mu2>0.001</mu2>
         <material>Gazebo/Black</material>
     </gazebo>
